File: part1_rc_servo/part1_rc_servo.kicad_sch (KiCad schematic)
At the start: 0 parts

Commit message: chore(part1): switch to A3, reposition blocks L→R, enlarge fonts; orthogonal routing; add rails bars; ensure servo on-page; re-export PNG/PDF/SVG
Co-authored-by: Amber Borjigin <aborjigin@users.noreply.github.com>
Other:
- note added: "5V (orange)"
- note added: "Common ground for ATX, UNO boards, rails, and servo"
- note added: "GND (brown)"
- note added: "GND to rails"
- note added: "LED bank: scaled pot value (LED_BANK1–3)"
- note added: "Limit wiper 0–3.3V"
- note added: "Power distribution"
- note added: "Signal (yellow)"
- note added: "W03 — Analog input 0–3.3V (AD_PORTW3)"
- note added: "Y06 — Digital output 0–3.3V (RC_PORTY06, Timer4)"
- note removed: "12V + GND in from ATX"
- note removed: "5V to servo (+)"
- note removed: "5V: orange (regulated 5V)"
- note removed: "Ends → 5V and GND rails"
- note removed: "Feeds UNO IO board"
- note removed: "GND to servo (−)"
- note removed: "GND: brown"
- note removed: "LED bank: displays scaled pot value (LED_BANK1–3)"
- note removed: "Limit wiper to 0–3.3V"
- note removed: "NOTE: Common ground between ATX supply, UNO boards, servo, and breadboard rails."
- note removed: "Signal: yellow"
- note removed: "W03 — Analog input 0–3.3V"
- note removed: "W03 → Analog input (AD_PORTW3) 0–3.3V"
- note removed: "Wiper → UNO W03"
- note removed: "Y06 — Digital output 0–3.3V"
- note removed: "Y06 → Servo signal (RC_PORTY06, Timer4)"
Changed lines of the file:
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@@
 (kicad_sch (version 20230121) (generator eeschema)
-   (paper "A4")
-   (title_block
-     (title "ECE118 Lab 3 — Part 1: Driving an RC Servo (Block Diagram)")
-     (company "UCSC ECE118 — Student: Amber")
-     (rev "A")
-   )
-   (polyline (pts (xy 20 40) (xy 80 40) (xy 80 85) (xy 20 85) (xy 20 40)) (stroke (width 0.6) (type solid)))
-   (text "ATX power supply" (at 25 45 0) (effects (font (size 3.5 3.5)) (justify left bottom)))
-   (text "Outputs: 12V, 5V, GND" (at 25 52 0) (effects (font (size 2.2 2.2)) (justify left bottom)))
-   (polyline (pts (xy 95 45) (xy 165 45) (xy 165 80) (xy 95 80) (xy 95 45)) (stroke (width 0.6) (type solid)))
-   (text "UNO power board" (at 100 50 0) (effects (font (size 3.2 3.2)) (justify left bottom)))
-   (text "12V + GND in from ATX" (at 100 57 0) (effects (font (size 2.2 2.2)) (justify left bottom)))
-   (text "Feeds UNO IO board" (at 100 63.5 0) (effects (font (size 2.2 2.2)) (justify left bottom)))
-   (polyline (pts (xy 95 95) (xy 165 95) (xy 165 160) (xy 95 160) (xy 95 95)) (stroke (width 0.6) (type solid)))
-   (text "UNO32 IO board" (at 100 100 0) (effects (font (size 3.2 3.2)) (justify left bottom)))
-   (text "W03 → Analog input (AD_PORTW3) 0–3.3V" (at 100 108 0) (effects (font (size 2.2 2.2)) (justify left bottom)))
-   (text "Y06 → Servo signal (RC_PORTY06, Timer4)" (at 100 114 0) (effects (font (size 2.2 2.2)) (justify left bottom)))
-   (text "LED bank: displays scaled pot value (LED_BANK1–3)" (at 100 120 0) (effects (font (size 2.0 2.0)) (justify left bottom)))
-   (polyline (pts (xy 185 45) (xy 280 45) (xy 280 160) (xy 185 160) (xy 185 45)) (stroke (width 0.6) (type solid)))
-   (text "Breadboard" (at 190 50 0) (effects (font (size 3.2 3.2)) (justify left bottom)))
-   (text "5V rail" (at 195 62 0) (effects (font (size 2.4 2.4)) (justify left bottom)))
-   (polyline (pts (xy 192 65) (xy 273 65)) (stroke (width 0.6) (type solid)))
-   (text "GND rail" (at 195 72 0) (effects (font (size 2.4 2.4)) (justify left bottom)))
-   (polyline (pts (xy 192 75) (xy 273 75)) (stroke (width 0.6) (type solid)))
-   (polyline (pts (xy 210 95) (xy 255 95) (xy 255 130) (xy 210 130) (xy 210 95)) (stroke (width 0.5) (type solid)))
-   (text "Potentiometer" (at 212 100 0) (effects (font (size 2.6 2.6)) (justify left bottom)))
-   (text "Ends → 5V and GND rails" (at 212 106 0) (effects (font (size 2.0 2.0)) (justify left bottom)))
-   (text "Wiper → UNO W03" (at 212 112 0) (effects (font (size 2.0 2.0)) (justify left bottom)))
-   (text "Limit wiper to 0–3.3V" (at 212 118 0) (effects (font (size 2.0 2.0)) (justify left bottom)))
-   (polyline (pts (xy 315 90) (xy 390 90) (xy 390 140) (xy 315 140) (xy 315 90)) (stroke (width 0.6) (type solid)))
-   (text "RC Servo" (at 320 95 0) (effects (font (size 3.2 3.2)) (justify left bottom)))
-   (text "Signal: yellow" (at 320 104 0) (effects (font (size 2.0 2.0)) (justify left bottom)))
-   (text "5V: orange (regulated 5V)" (at 320 110 0) (effects (font (size 2.0 2.0)) (justify left bottom)))
-   (text "GND: brown" (at 320 116 0) (effects (font (size 2.0 2.0)) (justify left bottom)))
-   (polyline (pts (xy 80 60) (xy 95 60)) (stroke (width 0.6) (type solid)))
-   (text "12V" (at 86 57 0) (effects (font (size 2.2 2.2)) (justify left bottom)))
-   (polyline (pts (xy 80 70) (xy 95 70)) (stroke (width 0.6) (type solid)))
-   (text "GND" (at 86 73 0) (effects (font (size 2.2 2.2)) (justify left bottom)))
-   (text "NOTE: Common ground between ATX supply, UNO boards,\nservo, and breadboard rails." (at 20 92 0) (effects (font (size 2.0 2.0)) (justify left bottom)))
-   (polyline (pts (xy 185 120) (xy 165 120)) (stroke (width 0.6) (type solid)))
-   (text "W03 — Analog input 0–3.3V" (at 142 123 0) (effects (font (size 2.2 2.2)) (justify left bottom)))
-   (polyline (pts (xy 210 120) (xy 185 120)) (stroke (width 0.6) (type solid)))
-   (polyline (pts (xy 210 100) (xy 192 65)) (stroke (width 0.6) (type solid)))
-   (polyline (pts (xy 210 125) (xy 192 75)) (stroke (width 0.6) (type solid)))
-   (text "5V rail" (at 196 62 0) (effects (font (size 2.0 2.0)) (justify left bottom)))
-   (text "GND rail" (at 196 78 0) (effects (font (size 2.0 2.0)) (justify left bottom)))
-   (polyline (pts (xy 80 55) (xy 185 55) (xy 185 65)) (stroke (width 0.6) (type solid)))
-   (text "5V (regulated)" (at 120 53 0) (effects (font (size 2.2 2.2)) (justify left bottom)))
-   (polyline (pts (xy 80 75) (xy 185 75)) (stroke (width 0.6) (type solid)))
-   (text "GND" (at 120 77 0) (effects (font (size 2.2 2.2)) (justify left bottom)))
-   (polyline (pts (xy 165 140) (xy 315 140)) (stroke (width 0.6) (type solid)))
-   (text "Y06 — Digital output 0–3.3V" (at 175 144 0) (effects (font (size 2.2 2.2)) (justify left bottom)))
-   (text "RC servo pulse ~1–2 ms, 50 ms period" (at 175 149 0) (effects (font (size 2.0 2.0)) (justify left bottom)))
-   (polyline (pts (xy 315 110) (xy 273 65)) (stroke (width 0.6) (type solid)))
-   (polyline (pts (xy 315 120) (xy 273 75)) (stroke (width 0.6) (type solid)))
-   (text "5V to servo (+)" (at 290 84 0) (effects (font (size 2.0 2.0)) (justify left bottom)))
-   (text "GND to servo (−)" (at 290 130 0) (effects (font (size 2.0 2.0)) (justify left bottom)))
-   (polyline (pts (xy 130 80) (xy 130 95)) (stroke (width 0.6) (type solid)))
-   (text "Power" (at 132 88 0) (effects (font (size 2.0 2.0)) (justify left bottom)))
- )
+  (paper "A3")
+  (title_block
+    (title "ECE118 Lab 3 — Part 1: Driving an RC Servo (Block Diagram)")
+    (company "UCSC ECE118 — Student: Amber")
+    (rev "B")
+  )
+  (polyline (pts (xy 20 70) (xy 90 70) (xy 90 130) (xy 20 130) (xy 20 70)) (stroke (width 0.6) (type solid)))
+  (text "ATX power supply" (at 25 75 0) (effects (font (size 5 5)) (justify left bottom)))
+  (text "Outputs: 12V, 5V, GND" (at 25 83 0) (effects (font (size 3 3)) (justify left bottom)))
+  (polyline (pts (xy 110 70) (xy 170 70) (xy 170 130) (xy 110 130) (xy 110 70)) (stroke (width 0.6) (type solid)))
+  (text "UNO power board" (at 115 75 0) (effects (font (size 5 5)) (justify left bottom)))
+  (text "Power distribution" (at 115 83 0) (effects (font (size 3 3)) (justify left bottom)))
+  (polyline (pts (xy 190 70) (xy 250 70) (xy 250 140) (xy 190 140) (xy 190 70)) (stroke (width 0.6) (type solid)))
+  (text "UNO32 IO board" (at 195 75 0) (effects (font (size 5 5)) (justify left bottom)))
+  (text "LED bank: scaled pot value (LED_BANK1–3)" (at 195 98 0) (effects (font (size 3 3)) (justify left bottom)))
+  (polyline (pts (xy 270 60) (xy 360 60) (xy 360 150) (xy 270 150) (xy 270 60)) (stroke (width 0.6) (type solid)))
+  (text "Breadboard" (at 275 65 0) (effects (font (size 5 5)) (justify left bottom)))
+  (polyline (pts (xy 370 100) (xy 410 100) (xy 410 145) (xy 370 145) (xy 370 100)) (stroke (width 0.6) (type solid)))
+  (text "RC Servo" (at 372 105 0) (effects (font (size 5 5)) (justify left bottom)))
+  (text "Signal (yellow)" (at 372 132 0) (effects (font (size 3 3)) (justify left bottom)))
+  (text "5V (orange)" (at 372 114 0) (effects (font (size 3 3)) (justify left bottom)))
+  (text "GND (brown)" (at 372 120 0) (effects (font (size 3 3)) (justify left bottom)))
+  (polyline (pts (xy 277 80) (xy 353 80)) (stroke (width 0.8) (type solid)))
+  (text "5V rail" (at 279 76 0) (effects (font (size 3 3)) (justify left bottom)))
+  (polyline (pts (xy 277 90) (xy 353 90)) (stroke (width 0.8) (type solid)))
+  (text "GND rail" (at 279 94 0) (effects (font (size 3 3)) (justify left bottom)))
+  (polyline (pts (xy 300 105) (xy 345 105) (xy 345 140) (xy 300 140) (xy 300 105)) (stroke (width 0.5) (type solid)))
+  (text "Potentiometer" (at 302 110 0) (effects (font (size 3 3)) (justify left bottom)))
+  (text "Limit wiper 0–3.3V" (at 302 116 0) (effects (font (size 3 3)) (justify left bottom)))
+  (polyline (pts (xy 90 90) (xy 110 90)) (stroke (width 0.6) (type solid)))
+  (text "12V" (at 94 86 0) (effects (font (size 3 3)) (justify left bottom)))
+  (polyline (pts (xy 90 110) (xy 110 110)) (stroke (width 0.6) (type solid)))
+  (text "GND" (at 94 114 0) (effects (font (size 3 3)) (justify left bottom)))
+  (polyline (pts (xy 90 72) (xy 270 72) (xy 270 80)) (stroke (width 0.6) (type solid)))
+  (text "5V (regulated)" (at 140 68 0) (effects (font (size 3 3)) (justify left bottom)))
+  (polyline (pts (xy 90 120) (xy 260 120) (xy 260 90) (xy 270 90)) (stroke (width 0.6) (type solid)))
+  (text "GND to rails" (at 140 122 0) (effects (font (size 3 3)) (justify left bottom)))
+  (polyline (pts (xy 170 100) (xy 190 100)) (stroke (width 0.6) (type solid)))
+  (text "Power" (at 173 96 0) (effects (font (size 3 3)) (justify left bottom)))
+  (polyline (pts (xy 305 105) (xy 305 80)) (stroke (width 0.6) (type solid)))
+  (polyline (pts (xy 305 140) (xy 305 90)) (stroke (width 0.6) (type solid)))
+  (polyline (pts (xy 322 122) (xy 260 122) (xy 260 120) (xy 190 120)) (stroke (width 0.6) (type solid)))
+  (text "W03 — Analog input 0–3.3V (AD_PORTW3)" (at 195 116 0) (effects (font (size 3 3)) (justify left bottom)))
+  (polyline (pts (xy 250 130) (xy 370 130)) (stroke (width 0.6) (type solid)))
+  (text "Y06 — Digital output 0–3.3V (RC_PORTY06, Timer4)" (at 195 135 0) (effects (font (size 3 3)) (justify left bottom)))
+  (text "RC servo pulse ~1–2 ms, 50 ms period" (at 195 141 0) (effects (font (size 3 3)) (justify left bottom)))
+  (polyline (pts (xy 353 80) (xy 370 80) (xy 370 110)) (stroke (width 0.6) (type solid)))
+  (polyline (pts (xy 353 90) (xy 385 90) (xy 385 115)) (stroke (width 0.6) (type solid)))
+  (text "Common ground for ATX, UNO boards, rails, and servo" (at 22 138 0) (effects (font (size 3 3)) (justify left bottom)))
+)

Commit message: refactor(part1): regenerate schematic via gen_part1.py; enforce ≥25mm gaps, no text/wire crossings; orthogonal routing; updated A3 exports (PNG/PDF/SVG)
Co-authored-by: Amber Borjigin <aborjigin@users.noreply.github.com>
Other:
- note added: "5V to servo (+)"
- note added: "GND to servo (−)"
- note removed: "5V (orange)"
- note removed: "GND (brown)"
- note removed: "Outputs: 12V, 5V, GND"
- note removed: "Power distribution"
- note removed: "Signal (yellow)"
Changed lines of the file:
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@@
     (title "ECE118 Lab 3 — Part 1: Driving an RC Servo (Block Diagram)")
     (company "UCSC ECE118 — Student: Amber")
-    (rev "B")
+    (rev "C")
   )
-  (polyline (pts (xy 20 70) (xy 90 70) (xy 90 130) (xy 20 130) (xy 20 70)) (stroke (width 0.6) (type solid)))
-  (text "ATX power supply" (at 25 75 0) (effects (font (size 5 5)) (justify left bottom)))
-  (text "Outputs: 12V, 5V, GND" (at 25 83 0) (effects (font (size 3 3)) (justify left bottom)))
-  (polyline (pts (xy 110 70) (xy 170 70) (xy 170 130) (xy 110 130) (xy 110 70)) (stroke (width 0.6) (type solid)))
-  (text "UNO power board" (at 115 75 0) (effects (font (size 5 5)) (justify left bottom)))
-  (text "Power distribution" (at 115 83 0) (effects (font (size 3 3)) (justify left bottom)))
-  (polyline (pts (xy 190 70) (xy 250 70) (xy 250 140) (xy 190 140) (xy 190 70)) (stroke (width 0.6) (type solid)))
-  (text "UNO32 IO board" (at 195 75 0) (effects (font (size 5 5)) (justify left bottom)))
-  (text "LED bank: scaled pot value (LED_BANK1–3)" (at 195 98 0) (effects (font (size 3 3)) (justify left bottom)))
-  (polyline (pts (xy 270 60) (xy 360 60) (xy 360 150) (xy 270 150) (xy 270 60)) (stroke (width 0.6) (type solid)))
-  (text "Breadboard" (at 275 65 0) (effects (font (size 5 5)) (justify left bottom)))
-  (polyline (pts (xy 370 100) (xy 410 100) (xy 410 145) (xy 370 145) (xy 370 100)) (stroke (width 0.6) (type solid)))
-  (text "RC Servo" (at 372 105 0) (effects (font (size 5 5)) (justify left bottom)))
-  (text "Signal (yellow)" (at 372 132 0) (effects (font (size 3 3)) (justify left bottom)))
-  (text "5V (orange)" (at 372 114 0) (effects (font (size 3 3)) (justify left bottom)))
-  (text "GND (brown)" (at 372 120 0) (effects (font (size 3 3)) (justify left bottom)))
-  (polyline (pts (xy 277 80) (xy 353 80)) (stroke (width 0.8) (type solid)))
-  (text "5V rail" (at 279 76 0) (effects (font (size 3 3)) (justify left bottom)))
-  (polyline (pts (xy 277 90) (xy 353 90)) (stroke (width 0.8) (type solid)))
-  (text "GND rail" (at 279 94 0) (effects (font (size 3 3)) (justify left bottom)))
-  (polyline (pts (xy 300 105) (xy 345 105) (xy 345 140) (xy 300 140) (xy 300 105)) (stroke (width 0.5) (type solid)))
-  (text "Potentiometer" (at 302 110 0) (effects (font (size 3 3)) (justify left bottom)))
-  (text "Limit wiper 0–3.3V" (at 302 116 0) (effects (font (size 3 3)) (justify left bottom)))
-  (polyline (pts (xy 90 90) (xy 110 90)) (stroke (width 0.6) (type solid)))
-  (text "12V" (at 94 86 0) (effects (font (size 3 3)) (justify left bottom)))
-  (polyline (pts (xy 90 110) (xy 110 110)) (stroke (width 0.6) (type solid)))
-  (text "GND" (at 94 114 0) (effects (font (size 3 3)) (justify left bottom)))
-  (polyline (pts (xy 90 72) (xy 270 72) (xy 270 80)) (stroke (width 0.6) (type solid)))
-  (text "5V (regulated)" (at 140 68 0) (effects (font (size 3 3)) (justify left bottom)))
-  (polyline (pts (xy 90 120) (xy 260 120) (xy 260 90) (xy 270 90)) (stroke (width 0.6) (type solid)))
-  (text "GND to rails" (at 140 122 0) (effects (font (size 3 3)) (justify left bottom)))
-  (polyline (pts (xy 170 100) (xy 190 100)) (stroke (width 0.6) (type solid)))
-  (text "Power" (at 173 96 0) (effects (font (size 3 3)) (justify left bottom)))
-  (polyline (pts (xy 305 105) (xy 305 80)) (stroke (width 0.6) (type solid)))
-  (polyline (pts (xy 305 140) (xy 305 90)) (stroke (width 0.6) (type solid)))
-  (polyline (pts (xy 322 122) (xy 260 122) (xy 260 120) (xy 190 120)) (stroke (width 0.6) (type solid)))
-  (text "W03 — Analog input 0–3.3V (AD_PORTW3)" (at 195 116 0) (effects (font (size 3 3)) (justify left bottom)))
-  (polyline (pts (xy 250 130) (xy 370 130)) (stroke (width 0.6) (type solid)))
-  (text "Y06 — Digital output 0–3.3V (RC_PORTY06, Timer4)" (at 195 135 0) (effects (font (size 3 3)) (justify left bottom)))
-  (text "RC servo pulse ~1–2 ms, 50 ms period" (at 195 141 0) (effects (font (size 3 3)) (justify left bottom)))
-  (polyline (pts (xy 353 80) (xy 370 80) (xy 370 110)) (stroke (width 0.6) (type solid)))
-  (polyline (pts (xy 353 90) (xy 385 90) (xy 385 115)) (stroke (width 0.6) (type solid)))
-  (text "Common ground for ATX, UNO boards, rails, and servo" (at 22 138 0) (effects (font (size 3 3)) (justify left bottom)))
+  (polyline (pts (xy 20.000 30.000) (xy 110.000 30.000) (xy 110.000 75.000) (xy 20.000 75.000) (xy 20.000 30.000)) (stroke (width 0.6) (type solid)))
+  (polyline (pts (xy 140.000 30.000) (xy 240.000 30.000) (xy 240.000 75.000) (xy 140.000 75.000) (xy 140.000 30.000)) (stroke (width 0.6) (type solid)))
+  (polyline (pts (xy 10.000 210.000) (xy 130.000 210.000) (xy 130.000 270.000) (xy 10.000 270.000) (xy 10.000 210.000)) (stroke (width 0.6) (type solid)))
+  (polyline (pts (xy 160.000 100.000) (xy 300.000 100.000) (xy 300.000 210.000) (xy 160.000 210.000) (xy 160.000 100.000)) (stroke (width 0.6) (type solid)))
+  (polyline (pts (xy 330.000 120.000) (xy 405.000 120.000) (xy 405.000 175.000) (xy 330.000 175.000) (xy 330.000 120.000)) (stroke (width 0.6) (type solid)))
+  (polyline (pts (xy 210.000 145.000) (xy 270.000 145.000) (xy 270.000 190.000) (xy 210.000 190.000) (xy 210.000 145.000)) (stroke (width 0.6) (type solid)))
+  (polyline (pts (xy 165.000 115.000) (xy 295.000 115.000)) (stroke (width 0.800) (type solid)))
+  (polyline (pts (xy 165.000 125.000) (xy 295.000 125.000)) (stroke (width 0.800) (type solid)))
+  (polyline (pts (xy 215.000 145.000) (xy 215.000 115.000)) (stroke (width 0.600) (type solid)))
+  (polyline (pts (xy 215.000 190.000) (xy 215.000 125.000)) (stroke (width 0.600) (type solid)))
+  (polyline (pts (xy 110.000 50.000) (xy 140.000 50.000)) (stroke (width 0.600) (type solid)))
+  (polyline (pts (xy 110.000 60.000) (xy 140.000 60.000)) (stroke (width 0.600) (type solid)))
+  (polyline (pts (xy 110.000 80.000) (xy 150.000 80.000) (xy 150.000 115.000) (xy 165.000 115.000)) (stroke (width 0.600) (type solid)))
+  (polyline (pts (xy 110.000 90.000) (xy 145.000 90.000) (xy 145.000 125.000) (xy 165.000 125.000)) (stroke (width 0.600) (type solid)))
+  (polyline (pts (xy 230.000 75.000) (xy 230.000 200.000) (xy 130.000 200.000) (xy 130.000 210.000)) (stroke (width 0.600) (type solid)))
+  (polyline (pts (xy 240.000 167.500) (xy 240.000 220.000) (xy 140.000 220.000) (xy 140.000 230.000) (xy 130.000 230.000)) (stroke (width 0.600) (type solid)))
+  (polyline (pts (xy 130.000 250.000) (xy 315.000 250.000) (xy 315.000 150.000) (xy 330.000 150.000)) (stroke (width 0.600) (type solid)))
+  (polyline (pts (xy 295.000 115.000) (xy 320.000 115.000) (xy 320.000 135.000) (xy 330.000 135.000)) (stroke (width 0.600) (type solid)))
+  (polyline (pts (xy 295.000 125.000) (xy 310.000 125.000) (xy 310.000 160.000) (xy 330.000 160.000)) (stroke (width 0.600) (type solid)))
+  (text "ATX power supply" (at 25.000 38.000 0) (effects (font (size 5.000 5.000)) (justify left bottom)))
+  (text "UNO power board" (at 145.000 38.000 0) (effects (font (size 5.000 5.000)) (justify left bottom)))
+  (text "UNO32 IO board" (at 15.000 220.000 0) (effects (font (size 5.000 5.000)) (justify left bottom)))
+  (text "Breadboard" (at 165.000 108.000 0) (effects (font (size 5.000 5.000)) (justify left bottom)))
+  (text "RC Servo" (at 334.000 128.000 0) (effects (font (size 5.000 5.000)) (justify left bottom)))
+  (text "Potentiometer" (at 232.000 157.000 0) (effects (font (size 3.000 3.000)) (justify left bottom)))
+  (text "Limit wiper 0–3.3V" (at 232.000 165.000 0) (effects (font (size 3.000 3.000)) (justify left bottom)))
+  (text "LED bank: scaled pot value (LED_BANK1–3)" (at 12.000 238.000 0) (effects (font (size 3.000 3.000)) (justify left bottom)))
+  (text "5V rail" (at 167.000 112.500 0) (effects (font (size 3.000 3.000)) (justify left bottom)))
+  (text "GND rail" (at 167.000 130.500 0) (effects (font (size 3.000 3.000)) (justify left bottom)))
+  (text "12V" (at 120.000 47.000 0) (effects (font (size 3.000 3.000)) (justify left bottom)))
+  (text "GND" (at 119.000 64.000 0) (effects (font (size 3.000 3.000)) (justify left bottom)))
+  (text "5V (regulated)" (at 120.000 77.000 0) (effects (font (size 3.000 3.000)) (justify left bottom)))
+  (text "GND to rails" (at 120.000 94.000 0) (effects (font (size 3.000 3.000)) (justify left bottom)))
+  (text "Power" (at 105.000 197.000 0) (effects (font (size 3.000 3.000)) (justify left bottom)))
+  (text "W03 — Analog input 0–3.3V (AD_PORTW3)" (at 142.000 218.000 0) (effects (font (size 3.000 3.000)) (justify left bottom)))
+  (text "Y06 — Digital output 0–3.3V (RC_PORTY06, Timer4)" (at 132.000 248.000 0) (effects (font (size 3.000 3.000)) (justify left bottom)))
+  (text "RC servo pulse ~1–2 ms, 50 ms period" (at 132.000 256.000 0) (effects (font (size 3.000 3.000)) (justify left bottom)))
+  (text "5V to servo (+)" (at 275.000 113.000 0) (effects (font (size 3.000 3.000)) (justify left bottom)))
+  (text "GND to servo (−)" (at 265.000 129.000 0) (effects (font (size 3.000 3.000)) (justify left bottom)))
+  (text "Common ground for ATX, UNO boards, rails, and servo" (at 25.000 285.000 0) (effects (font (size 3.000 3.000)) (justify left bottom)))
 )
