File: part1_rc_servo/part1_rc_servo.kicad_sch (KiCad schematic)
At the start: 0 parts

Commit message: fix(part1): regenerate Rev D with no dangling ends, no wires through blocks; pot taps + wiper per spec; servo entry labels; A3 clean spacing; re-export PNG/PDF/SVG
Co-authored-by: Amber Borjigin <aborjigin@users.noreply.github.com>
Other:
- note added: "5V (orange) — max 5V, regulated"
- note added: "BB 5V rail"
- note added: "BB GND rail"
- note added: "GND (brown)"
- note added: "Signal (yellow)"
- note removed: "5V rail"
- note removed: "5V to servo (+)"
- note removed: "GND rail"
- note removed: "GND to servo (−)"
Changed lines of the file:
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@@
   (polyline (pts (xy 165.000 115.000) (xy 295.000 115.000)) (stroke (width 0.800) (type solid)))
   (polyline (pts (xy 165.000 125.000) (xy 295.000 125.000)) (stroke (width 0.800) (type solid)))
-  (polyline (pts (xy 215.000 145.000) (xy 215.000 115.000)) (stroke (width 0.600) (type solid)))
-  (polyline (pts (xy 215.000 190.000) (xy 215.000 125.000)) (stroke (width 0.600) (type solid)))
+  (polyline (pts (xy 218.000 115.000) (xy 218.000 145.000)) (stroke (width 0.600) (type solid)))
+  (polyline (pts (xy 250.000 125.000) (xy 250.000 145.000)) (stroke (width 0.600) (type solid)))
   (polyline (pts (xy 110.000 50.000) (xy 140.000 50.000)) (stroke (width 0.600) (type solid)))
   (polyline (pts (xy 110.000 60.000) (xy 140.000 60.000)) (stroke (width 0.600) (type solid)))
-  (polyline (pts (xy 110.000 80.000) (xy 150.000 80.000) (xy 150.000 115.000) (xy 165.000 115.000)) (stroke (width 0.600) (type solid)))
-  (polyline (pts (xy 110.000 90.000) (xy 145.000 90.000) (xy 145.000 125.000) (xy 165.000 125.000)) (stroke (width 0.600) (type solid)))
-  (polyline (pts (xy 230.000 75.000) (xy 230.000 200.000) (xy 130.000 200.000) (xy 130.000 210.000)) (stroke (width 0.600) (type solid)))
-  (polyline (pts (xy 240.000 167.500) (xy 240.000 220.000) (xy 140.000 220.000) (xy 140.000 230.000) (xy 130.000 230.000)) (stroke (width 0.600) (type solid)))
-  (polyline (pts (xy 130.000 250.000) (xy 315.000 250.000) (xy 315.000 150.000) (xy 330.000 150.000)) (stroke (width 0.600) (type solid)))
-  (polyline (pts (xy 295.000 115.000) (xy 320.000 115.000) (xy 320.000 135.000) (xy 330.000 135.000)) (stroke (width 0.600) (type solid)))
-  (polyline (pts (xy 295.000 125.000) (xy 310.000 125.000) (xy 310.000 160.000) (xy 330.000 160.000)) (stroke (width 0.600) (type solid)))
+  (polyline (pts (xy 110.000 65.000) (xy 115.000 65.000) (xy 115.000 80.000) (xy 150.000 80.000) (xy 150.000 115.000) (xy 165.000 115.000)) (stroke (width 0.600) (type solid)))
+  (polyline (pts (xy 110.000 70.000) (xy 115.000 70.000) (xy 115.000 90.000) (xy 145.000 90.000) (xy 145.000 125.000) (xy 165.000 125.000)) (stroke (width 0.600) (type solid)))
+  (polyline (pts (xy 190.000 75.000) (xy 190.000 79.000) (xy 130.000 79.000) (xy 130.000 202.000) (xy 130.000 202.000) (xy 130.000 210.000)) (stroke (width 0.600) (type solid)))
+  (polyline (pts (xy 270.000 167.500) (xy 275.000 167.500) (xy 275.000 205.000) (xy 159.000 205.000) (xy 159.000 218.000) (xy 160.000 218.000) (xy 140.000 218.000) (xy 140.000 232.000) (xy 130.000 232.000)) (stroke (width 0.600) (type solid)))
+  (polyline (pts (xy 130.000 252.000) (xy 312.000 252.000) (xy 312.000 150.000) (xy 330.000 150.000)) (stroke (width 0.600) (type solid)))
+  (polyline (pts (xy 295.000 115.000) (xy 300.000 115.000) (xy 308.000 115.000) (xy 308.000 135.000) (xy 330.000 135.000)) (stroke (width 0.600) (type solid)))
+  (polyline (pts (xy 295.000 125.000) (xy 300.000 125.000) (xy 316.000 125.000) (xy 316.000 160.000) (xy 330.000 160.000)) (stroke (width 0.600) (type solid)))
   (text "ATX power supply" (at 25.000 38.000 0) (effects (font (size 5.000 5.000)) (justify left bottom)))
   (text "UNO power board" (at 145.000 38.000 0) (effects (font (size 5.000 5.000)) (justify left bottom)))
@@
   (text "Potentiometer" (at 232.000 157.000 0) (effects (font (size 3.000 3.000)) (justify left bottom)))
   (text "Limit wiper 0–3.3V" (at 232.000 165.000 0) (effects (font (size 3.000 3.000)) (justify left bottom)))
-  (text "LED bank: scaled pot value (LED_BANK1–3)" (at 12.000 238.000 0) (effects (font (size 3.000 3.000)) (justify left bottom)))
-  (text "5V rail" (at 167.000 112.500 0) (effects (font (size 3.000 3.000)) (justify left bottom)))
-  (text "GND rail" (at 167.000 130.500 0) (effects (font (size 3.000 3.000)) (justify left bottom)))
+  (text "LED bank: scaled pot value (LED_BANK1–3)" (at 16.000 238.000 0) (effects (font (size 3.000 3.000)) (justify left bottom)))
+  (text "BB 5V rail" (at 167.000 112.500 0) (effects (font (size 3.000 3.000)) (justify left bottom)))
+  (text "BB GND rail" (at 167.000 130.500 0) (effects (font (size 3.000 3.000)) (justify left bottom)))
   (text "12V" (at 120.000 47.000 0) (effects (font (size 3.000 3.000)) (justify left bottom)))
   (text "GND" (at 119.000 64.000 0) (effects (font (size 3.000 3.000)) (justify left bottom)))
-  (text "5V (regulated)" (at 120.000 77.000 0) (effects (font (size 3.000 3.000)) (justify left bottom)))
-  (text "GND to rails" (at 120.000 94.000 0) (effects (font (size 3.000 3.000)) (justify left bottom)))
-  (text "Power" (at 105.000 197.000 0) (effects (font (size 3.000 3.000)) (justify left bottom)))
-  (text "W03 — Analog input 0–3.3V (AD_PORTW3)" (at 142.000 218.000 0) (effects (font (size 3.000 3.000)) (justify left bottom)))
-  (text "Y06 — Digital output 0–3.3V (RC_PORTY06, Timer4)" (at 132.000 248.000 0) (effects (font (size 3.000 3.000)) (justify left bottom)))
-  (text "RC servo pulse ~1–2 ms, 50 ms period" (at 132.000 256.000 0) (effects (font (size 3.000 3.000)) (justify left bottom)))
-  (text "5V to servo (+)" (at 275.000 113.000 0) (effects (font (size 3.000 3.000)) (justify left bottom)))
-  (text "GND to servo (−)" (at 265.000 129.000 0) (effects (font (size 3.000 3.000)) (justify left bottom)))
+  (text "5V (regulated)" (at 260.000 121.000 0) (effects (font (size 3.000 3.000)) (justify left bottom)))
+  (text "GND to rails" (at 260.000 137.000 0) (effects (font (size 3.000 3.000)) (justify left bottom)))
+  (text "Power" (at 132.000 140.500 0) (effects (font (size 3.000 3.000)) (justify left bottom)))
+  (text "W03 — Analog input 0–3.3V (AD_PORTW3)" (at 150.000 226.000 0) (effects (font (size 3.000 3.000)) (justify left bottom)))
+  (text "Y06 — Digital output 0–3.3V (RC_PORTY06, Timer4)" (at 132.000 250.000 0) (effects (font (size 3.000 3.000)) (justify left bottom)))
+  (text "RC servo pulse ~1–2 ms, 50 ms period" (at 132.000 258.000 0) (effects (font (size 3.000 3.000)) (justify left bottom)))
+  (text "5V (orange) — max 5V, regulated" (at 332.000 133.000 0) (effects (font (size 3.000 3.000)) (justify left bottom)))
+  (text "GND (brown)" (at 332.000 158.000 0) (effects (font (size 3.000 3.000)) (justify left bottom)))
+  (text "Signal (yellow)" (at 332.000 148.000 0) (effects (font (size 3.000 3.000)) (justify left bottom)))
   (text "Common ground for ATX, UNO boards, rails, and servo" (at 25.000 285.000 0) (effects (font (size 3.000 3.000)) (justify left bottom)))
 )
