File: part1_rc_servo/part1_rc_servo.kicad_sch (KiCad schematic)
At the start: 0 parts

Commit message: fix(part1): Rev F schematic and exports per exact grid layout; verified single allowed crossing (wiper over GND rail) and no text/line collisions
Co-authored-by: Amber Borjigin <aborjigin@users.noreply.github.com>
Other:
- note added: "5 V regulated, max 5 V"
- note added: "5V (orange)"
- note added: "Common ground: ATX, UNO boards, breadboard rails, and servo"
- note added: "LED bank: scaled pot value (LED_BANK1-3)"
- note added: "W03 analog in, 0-3.3 V"
- note added: "W03: analog in (AD_PORTW3)"
- note added: "Y06 digital out, 0-3.3 V"
- note added: "Y06: servo out (RC_PORTY06, Timer4)"
- note added: "pulse 1-2 ms every 50 ms"
- note added: "wiper 0-3.3 V"
- note removed: "5V (orange) — max 5V, regulated"
- note removed: "Common ground for ATX, UNO boards, rails, and servo"
- note removed: "GND to rails"
- note removed: "LED bank: scaled pot value (LED_BANK1–3)"
- note removed: "Limit wiper 0–3.3V"
- note removed: "RC servo pulse ~1–2 ms, 50 ms period"
- note removed: "W03 — Analog input 0–3.3V (AD_PORTW3)"
- note removed: "Y06 — Digital output 0–3.3V (RC_PORTY06, Timer4)"
